Commit message: The 7DOF robot is up and shown in gazebo

File: Project_5_Building_A_ROS_NODE_With_Gazebo/resources/mastering_ros_robot_description_pkg/urdf/seven_dof_arm.xacro (robot description, xacro)
@@ -11,44 +11,44 @@
         <color rgba="1.0 1.0 1.0 1.0"/>
     </material>
-  <property name="deg_to_rad" value="0.01745329251994329577"/>
+  <xacro:property name="deg_to_rad" value="0.01745329251994329577"/>
   <!-- Constants -->
-  <property name="M_SCALE" value="0.001 0.001 0.001"/>
-  <property name="M_PI" value="3.14159"/>
+  <xacro:property name="M_SCALE" value="0.001 0.001 0.001"/>
+  <xacro:property name="M_PI" value="3.14159"/>
   <!-- Shoulder pan link properties -->
-  <property name="shoulder_pan_width" value="0.04" />
-  <property name="shoulder_pan_len" value="0.08" />
+  <xacro:property name="shoulder_pan_width" value="0.04" />
+  <xacro:property name="shoulder_pan_len" value="0.08" />
   <!-- Shoulder pitch link properties -->
-  <property name="shoulder_pitch_len" value="0.14" />
-  <property name="shoulder_pitch_width" value="0.04" />
-  <property name="shoulder_pitch_height" value="0.04" />
+  <xacro:property name="shoulder_pitch_len" value="0.14" />
+  <xacro:property name="shoulder_pitch_width" value="0.04" />
+  <xacro:property name="shoulder_pitch_height" value="0.04" />
   <!-- Elbow roll link properties -->
-  <property name="elbow_roll_width" value="0.02" />
-  <property name="elbow_roll_len" value="0.06" />
+  <xacro:property name="elbow_roll_width" value="0.02" />
+  <xacro:property name="elbow_roll_len" value="0.06" />
   <!-- Elbow pitch link properties -->
-  <property name="elbow_pitch_len" value="0.22" />
-  <property name="elbow_pitch_width" value="0.04" />
-  <property name="elbow_pitch_height" value="0.04" />
+  <xacro:property name="elbow_pitch_len" value="0.22" />
+  <xacro:property name="elbow_pitch_width" value="0.04" />
+  <xacro:property name="elbow_pitch_height" value="0.04" />
   <!-- Wrist roll link properties -->
-  <property name="wrist_roll_width" value="0.02" />
-  <property name="wrist_roll_len" value="0.04" />
+  <xacro:property name="wrist_roll_width" value="0.02" />
+  <xacro:property name="wrist_roll_len" value="0.04" />
   <!-- wrist pitch link properties -->
-  <property name="wrist_pitch_len" value="0.06" />
-  <property name="wrist_pitch_width" value="0.04" />
-  <property name="wrist_pitch_height" value="0.04" />
+  <xacro:property name="wrist_pitch_len" value="0.06" />
+  <xacro:property name="wrist_pitch_width" value="0.04" />
+  <xacro:property name="wrist_pitch_height" value="0.04" />
   <!-- Gripper roll link properties -->
-  <property name="gripper_roll_width" value="0.04" />
-  <property name="gripper_roll_len" value="0.02" />
+  <xacro:property name="gripper_roll_width" value="0.04" />
+  <xacro:property name="gripper_roll_len" value="0.02" />
   <!-- Left gripper -->
-  <property name="left_gripper_len" value="0.08" />
-  <property name="left_gripper_width" value="0.01" />
-  <property name="left_gripper_height" value="0.01" />
+  <xacro:property name="left_gripper_len" value="0.08" />
+  <xacro:property name="left_gripper_width" value="0.01" />
+  <xacro:property name="left_gripper_height" value="0.01" />
   <!-- Right gripper -->
-  <property name="right_gripper_len" value="0.08" />
-  <property name="right_gripper_width" value="0.01" />
-  <property name="right_gripper_height" value="0.01" />
+  <xacro:property name="right_gripper_len" value="0.08" />
+  <xacro:property name="right_gripper_width" value="0.01" />
+  <xacro:property name="right_gripper_height" value="0.01" />
   <!-- Right gripper -->
-  <property name="grasp_frame_len" value="0.02" />
-  <property name="grasp_frame_width" value="0.02" />
-  <property name="grasp_frame_height" value="0.02" />
+  <xacro:property name="grasp_frame_len" value="0.02" />
+  <xacro:property name="grasp_frame_width" value="0.02" />
+  <xacro:property name="grasp_frame_height" value="0.02" />
    <xacro:macro name="inertial_matrix" params="mass">
       <inertial>
